File: SOIC-8 Breakout/SOIC-8 Breakout.kicad_sch (KiCad schematic)
At the start: 19 parts, among them J1 IO, J2 IO, J3 ANC, J4 ANC, U1 LM555xM

Commit message: Updated Files
Parts:
- removed C1, C10, C11, C12, C13, C14, C2, C3, C4, C5, C6, C7, C8, C9: C, Capacitor_SMD:C_0603_1608Metric, symbol Device:C_Small
- removed J1, J2: IO, Connector_PinHeader_2.54mm:PinHeader_1x04_P2.54mm_Vertical, symbol Connector_Generic:Conn_01x04
- removed J3, J4: ANC, Connector_PinHeader_2.54mm:PinHeader_1x01_P2.54mm_Vertical, symbol Connector_Generic:Conn_01x01
- removed U1: LM555xM, Package_SO:SOIC-8_3.9x4.9mm_P1.27mm, symbol Timer:LM555xM
