File: SOIC-8 Breakout/SOIC-8 Breakout.kicad_pcb (KiCad board)
At the start: 2 copper layers, 18.5 x 11.5 mm, 19 parts, among them J1 IO, J2 IO, J3 ANC, J4 ANC, U1 LM555xM

Commit message: Updated Files
Parts:
- removed C1, C10, C11, C12, C13, C14, C2, C3, C4, C5, C6, C7, C8, C9: C, Capacitor_SMD:C_0603_1608Metric
- removed J1, J2: IO, Connector_PinHeader_2.54mm:PinHeader_1x04_P2.54mm_Vertical
- removed J3, J4: ANC, Connector_PinHeader_2.54mm:PinHeader_1x01_P2.54mm_Vertical
- removed U1: LM555xM, Package_SO:SOIC-8_3.9x4.9mm_P1.27mm
- added REF**: C_0805_2012Metric, Capacitor_SMD:C_0805_2012Metric, F.Cu at (144.8, 104.1)
- added REF**: C_0805_2012Metric, Capacitor_SMD:C_0805_2012Metric, F.Cu at (147.3, 104.1)
- added REF**: C_0603_1608Metric, Capacitor_SMD:C_0603_1608Metric, F.Cu at (153.5, 105.4)
- added REF**: SOIC-8_3.9x4.9mm_P1.27mm, Package_SO:SOIC-8_3.9x4.9mm_P1.27mm, F.Cu at (152.4, 101.6)
- added REF**: C_0603_1608Metric, Capacitor_SMD:C_0603_1608Metric, F.Cu at (157.5, 99.1)
- added REF**: C_0603_1608Metric, Capacitor_SMD:C_0603_1608Metric, F.Cu at (157.5, 101.6)
- added REF**: C_1206_3216Metric, Capacitor_SMD:C_1206_3216Metric, F.Cu at (172.8, 101.1)
- added REF**: C_0805_2012Metric, Capacitor_SMD:C_0805_2012Metric, F.Cu at (147.3, 101.6)
- added REF**: C_0805_2012Metric, Capacitor_SMD:C_0805_2012Metric, F.Cu at (144.8, 99.1)
- added REF**: C_0805_2012Metric, Capacitor_SMD:C_0805_2012Metric, F.Cu at (147.3, 99.1)
- added REF**: C_0603_1608Metric, Capacitor_SMD:C_0603_1608Metric, F.Cu at (160.0, 104.1)
- added REF**: C_0402_1005Metric, Capacitor_SMD:C_0402_1005Metric, F.Cu at (166.4, 100.8)
- added REF**: C_0603_1608Metric, Capacitor_SMD:C_0603_1608Metric, F.Cu at (160.0, 99.1)
- added REF**: C_0805_2012Metric, Capacitor_SMD:C_0805_2012Metric, F.Cu at (168.5, 101.0)
- added REF**: C_0603_1608Metric, Capacitor_SMD:C_0603_1608Metric, F.Cu at (164.1, 101.1)
- added REF**: C_0603_1608Metric, Capacitor_SMD:C_0603_1608Metric, F.Cu at (157.5, 104.1)
Routing:
- net Net-(C11-Pad2): track 7.92 -> 0.00 mm
- net Net-(C10-Pad2): track 7.92 -> 0.00 mm
- net Net-(C1-Pad2): track 7.92 -> 0.00 mm
- net Net-(C4-Pad2): track 7.92 -> 0.00 mm
- net Net-(C2-Pad2): track 7.24 -> 0.00 mm
- net Net-(C3-Pad2): track 7.24 -> 0.00 mm
- net Net-(C12-Pad2): track 7.24 -> 0.00 mm
- net Net-(C10-Pad1): track 7.24 -> 0.00 mm
- net GND: track 3.93 -> 0.00 mm, vias 4 -> 0
- added copper zone on B.Cu, net (none)
- added copper zone on F.Cu, net (none)
- removed copper zone on B.Cu, net GND
- removed copper zone on F.Cu, net GND
Other:
- board size 18.5 x 11.5 mm -> 18 x 15.4 mm

Commit message: Updated Files
Parts:
- removed the REF** at (144.8, 104.1)
- removed the REF** at (147.3, 104.1)
- removed the REF** at (153.5, 105.4)
- removed the REF** at (157.5, 99.1)
- removed the REF** at (157.5, 101.6)
- removed the REF** at (172.8, 101.1)
- removed the REF** at (147.3, 101.6)
- removed the REF** at (144.8, 99.1)
- removed the REF** at (147.3, 99.1)
- removed the REF** at (160.0, 104.1)
- removed the REF** at (166.4, 100.8)
- removed the REF** at (160.0, 99.1)
- removed the REF** at (168.5, 101.0)
- removed the REF** at (164.1, 101.1)
- removed the REF** at (157.5, 104.1)
- added REF**: MSOP-8_3x3mm_P0.65mm, Package_SO:MSOP-8_3x3mm_P0.65mm, B.Cu at (152.4, 101.6)
- moved REF** 0.13 mm to (152.5, 101.6)

Commit message: Updated Files
Parts:
- removed REF**: SOIC-8_3.9x4.9mm_P1.27mm, Package_SO:SOIC-8_3.9x4.9mm_P1.27mm
- removed REF**: MSOP-8_3x3mm_P0.65mm, Package_SO:MSOP-8_3x3mm_P0.65mm
Changed lines of the file:
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@@
   )
   (net 0 "")
-  (footprint "Package_SO:SOIC-8_3.9x4.9mm_P1.27mm" (layer "F.Cu")
-    (at 152.527 101.6)
-    (descr "SOIC, 8 Pin (JEDEC MS-012AA, https://www.analog.com/media/en/package-pcb-resources/package/pkg_pdf/soic_narrow-r/r_8.pdf), generated with kicad-footprint-generator ipc_gullwing_generator.py")
-    (tags "SOIC SO")
-    (attr smd)
-    (fp_text reference "REF**" (at 0 -3.4) (layer "F.SilkS") hide
-      (effects (font (size 1 1) (thickness 0.15)))
-    )
-    (fp_text value "SOIC-8_3.9x4.9mm_P1.27mm" (at 0 3.4) (layer "F.Fab")
-      (effects (font (size 1 1) (thickness 0.15)))
-    )
-    (fp_text user "${REFERENCE}" (at 0 0) (layer "F.Fab")
-      (effects (font (size 0.98 0.98) (thickness 0.15)))
-    )
-    (model "${KICAD6_3DMODEL_DIR}/Package_SO.3dshapes/SOIC-8_3.9x4.9mm_P1.27mm.wrl"
-      (offset (xyz 0 0 0))
-      (scale (xyz 1 1 1))
-      (rotate (xyz 0 0 0))
-    )
-  )
-  (footprint "Package_SO:MSOP-8_3x3mm_P0.65mm" (layer "B.Cu")
-    (at 152.4 101.6 180)
-    (descr "MSOP, 8 Pin (https://www.jedec.org/system/files/docs/mo-187F.pdf variant AA), generated with kicad-footprint-generator ipc_gullwing_generator.py")
-    (tags "MSOP SO")
-    (attr smd)
-    (fp_text reference "REF**" (at 0 2.45) (layer "B.SilkS") hide
-      (effects (font (size 1 1) (thickness 0.15)) (justify mirror))
-    )
-    (fp_text value "MSOP-8_3x3mm_P0.65mm" (at 0 -2.45) (layer "B.Fab")
-      (effects (font (size 1 1) (thickness 0.15)) (justify mirror))
-    )
-    (model "${KICAD6_3DMODEL_DIR}/Package_SO.3dshapes/MSOP-8_3x3mm_P0.65mm.wrl"
-      (offset (xyz 0 0 0))
-      (scale (xyz 1 1 1))
-      (rotate (xyz 0 0 0))
-    )
-  )
   (gr_rect (start 143.383 93.853) (end 161.417 109.22) (layer "Edge.Cuts") (width 0.1) (fill none))
   (zone (net 0) (net_name "") (layer "F.Cu") (hatch edge 0.508)

Commit message: Updated Files
Parts:
- added REF**: SOIC-8_3.9x4.9mm_P1.27mm, Package_SO:SOIC-8_3.9x4.9mm_P1.27mm, F.Cu at (152.4, 101.6)
- added REF**: MSOP-8_3x3mm_P0.65mm, Package_SO:MSOP-8_3x3mm_P0.65mm, B.Cu at (152.4, 101.6)

Commit message: Updated files
Parts:
- added REF**: C_0402_1005Metric, Capacitor_SMD:C_0402_1005Metric, B.Cu at (151.3, 105.4)
- added REF**: C_0603_1608Metric, Capacitor_SMD:C_0603_1608Metric, B.Cu at (153.5, 97.8)
- added REF**: C_0402_1005Metric, Capacitor_SMD:C_0402_1005Metric, B.Cu at (147.3, 104.1)
- added REF**: C_0402_1005Metric, Capacitor_SMD:C_0402_1005Metric, B.Cu at (144.8, 99.1)
- added REF**: C_0603_1608Metric, Capacitor_SMD:C_0603_1608Metric, B.Cu at (160.0, 99.1)
- added REF**: C_0603_1608Metric, Capacitor_SMD:C_0603_1608Metric, B.Cu at (157.5, 99.1)
- added REF**: C_0402_1005Metric, Capacitor_SMD:C_0402_1005Metric, B.Cu at (144.8, 104.1)
- added REF**: C_0402_1005Metric, Capacitor_SMD:C_0402_1005Metric, B.Cu at (147.3, 101.6)
- added REF**: C_0603_1608Metric, Capacitor_SMD:C_0603_1608Metric, B.Cu at (157.5, 104.1)
- added REF**: C_0603_1608Metric, Capacitor_SMD:C_0603_1608Metric, B.Cu at (160.0, 104.1)
- added REF**: C_0603_1608Metric, Capacitor_SMD:C_0603_1608Metric, B.Cu at (157.5, 101.6)
- added REF**: C_0402_1005Metric, Capacitor_SMD:C_0402_1005Metric, B.Cu at (151.3, 97.8)
- added REF**: C_0603_1608Metric, Capacitor_SMD:C_0603_1608Metric, B.Cu at (153.5, 105.4)
- added REF**: C_0402_1005Metric, Capacitor_SMD:C_0402_1005Metric, B.Cu at (147.3, 99.1)
