File: SOT23 Breakout/SOT23 Breakout.kicad_sch (KiCad schematic)
At the start: 8 parts, among them J1 IO, J2 IO, J3 ANC, J4 ANC, Q1 NMOS, Q2 NMOS, Q3 NMOS, Q4 NMOS

Commit message: Updated Files
Parts:
- removed J1, J2: IO, Connector_PinHeader_2.54mm:PinHeader_1x06_P2.54mm_Vertical, symbol Connector_Generic:Conn_01x06
- removed J3, J4: ANC, Connector_PinHeader_2.54mm:PinHeader_1x01_P2.54mm_Vertical, symbol Connector_Generic:Conn_01x01
- removed Q1, Q2, Q3, Q4: NMOS, Package_TO_SOT_SMD:SOT-23, symbol Device:Q_NMOS_GDS
Connections:
- no-connect marks 2 -> 0
