File: SOT23 Breakout/SOT23 Breakout.kicad_pcb (KiCad board)
At the start: 2 copper layers, 17.5 x 10 mm, 8 parts, among them J1 IO, J2 IO, J3 ANC, J4 ANC, Q1 NMOS, Q2 NMOS, Q3 NMOS, Q4 NMOS

Commit message: Updated Files
Parts:
- removed J1, J2: IO, Connector_PinHeader_2.54mm:PinHeader_1x06_P2.54mm_Vertical
- removed J3, J4: ANC, Connector_PinHeader_2.54mm:PinHeader_1x01_P2.54mm_Vertical
- removed Q1, Q2, Q3, Q4: NMOS, Package_TO_SOT_SMD:SOT-23
- added REF**: C_0603_1608Metric, Capacitor_SMD:C_0603_1608Metric, F.Cu at (139.7, 99.1)
- added REF**: C_0603_1608Metric, Capacitor_SMD:C_0603_1608Metric, F.Cu at (144.8, 99.1)
- added REF**: SOT-23, Package_TO_SOT_SMD:SOT-23, F.Cu at (139.7, 101.6)
- added REF**: SOT-23, Package_TO_SOT_SMD:SOT-23, F.Cu at (144.8, 101.6)
- added REF**: C_0603_1608Metric, Capacitor_SMD:C_0603_1608Metric, F.Cu at (142.2, 99.1)
- added REF**: C_0805_2012Metric, Capacitor_SMD:C_0805_2012Metric, F.Cu at (144.8, 104.8)
- added REF**: C_0805_2012Metric, Capacitor_SMD:C_0805_2012Metric, F.Cu at (147.3, 104.8)
- added REF**: C_0805_2012Metric, Capacitor_SMD:C_0805_2012Metric, F.Cu at (139.7, 104.8)
- added REF**: C_0603_1608Metric, Capacitor_SMD:C_0603_1608Metric, F.Cu at (147.3, 99.1)
- added REF**: SOT-23, Package_TO_SOT_SMD:SOT-23, F.Cu at (154.9, 101.6)
- added REF**: SOT-23, Package_TO_SOT_SMD:SOT-23, F.Cu at (149.9, 101.6)
- added REF**: C_0805_2012Metric, Capacitor_SMD:C_0805_2012Metric, F.Cu at (154.9, 104.8)
- added REF**: C_0805_2012Metric, Capacitor_SMD:C_0805_2012Metric, F.Cu at (142.2, 104.8)
- added REF**: C_0805_2012Metric, Capacitor_SMD:C_0805_2012Metric, F.Cu at (152.4, 104.8)
- added REF**: C_0603_1608Metric, Capacitor_SMD:C_0603_1608Metric, F.Cu at (152.4, 99.1)
- added REF**: C_0603_1608Metric, Capacitor_SMD:C_0603_1608Metric, F.Cu at (154.9, 99.1)
- added REF**: C_0603_1608Metric, Capacitor_SMD:C_0603_1608Metric, F.Cu at (149.9, 99.1)
- added REF**: C_0805_2012Metric, Capacitor_SMD:C_0805_2012Metric, F.Cu at (149.9, 104.8)
Routing:
- net Net-(Q1-Pad3): track 3.68 -> 0.00 mm
- net Net-(Q4-Pad3): track 3.56 -> 0.00 mm
- net Net-(J2-Pad2): track 3.39 -> 0.00 mm
- net Net-(Q3-Pad2): track 3.27 -> 0.00 mm
- net Net-(J2-Pad5): track 3.14 -> 0.00 mm
- net Net-(Q3-Pad3): track 3.13 -> 0.00 mm
- net Net-(J2-Pad3): track 3.13 -> 0.00 mm
- net Net-(Q1-Pad2): track 3.02 -> 0.00 mm
- net Net-(Q2-Pad3): track 3.01 -> 0.00 mm
- net Net-(Q3-Pad1): track 3.01 -> 0.00 mm
- net Net-(J2-Pad6): track 2.99 -> 0.00 mm
- net Net-(Q1-Pad1): track 2.87 -> 0.00 mm
- added copper zone on F.Cu, net (none)
Other:
- board size 17.5 x 10 mm -> 20.6 x 10.4 mm

Commit message: Updated Files
Parts:
- removed REF** (x7): C_0603_1608Metric, Capacitor_SMD:C_0603_1608Metric
- removed REF** (x4): SOT-23, Package_TO_SOT_SMD:SOT-23
- removed REF** (x7): C_0805_2012Metric, Capacitor_SMD:C_0805_2012Metric

Commit message: Updated Files
Other:
- board size 20.6 x 10.4 mm -> 20.6 x 15.5 mm
Changed lines of the file:
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@@
   )
   (net 0 "")
-  (gr_rect (start 137.033 96.393) (end 157.607 106.807) (layer "Edge.Cuts") (width 0.1) (fill none))
+  (gr_rect (start 137.033 93.853) (end 157.607 109.347) (layer "Edge.Cuts") (width 0.1) (fill none))
+  (zone (net 0) (net_name "") (layer "F.Cu") (hatch edge 0.508)
+    (connect_pads (clearance 0.127))
+    (min_thickness 0.254) (filled_areas_thickness no)
+    (fill yes (thermal_gap 0.508) (thermal_bridge_width 0.508))
+    (polygon
+      (pts
+        (xy 154.813 109.093)
+        (xy 152.527 109.093)
+        (xy 152.527 106.807)
+        (xy 154.813 106.807)
+      )
+    )
+  )
   (zone (net 0) (net_name "") (layer "F.Cu") (hatch edge 0.508)
     (connect_pads yes (clearance 0.127))
@@
   )
   (zone (net 0) (net_name "") (layer "F.Cu") (hatch edge 0.508)
+    (connect_pads (clearance 0.127))
+    (min_thickness 0.254) (filled_areas_thickness no)
+    (fill yes (thermal_gap 0.508) (thermal_bridge_width 0.508))
+    (polygon
+      (pts
+        (xy 149.733 109.093)
+        (xy 147.447 109.093)
+        (xy 147.447 106.807)
+        (xy 149.733 106.807)
+      )
+    )
+  )
+  (zone (net 0) (net_name "") (layer "F.Cu") (hatch edge 0.508)
+    (connect_pads (clearance 0.127))
+    (min_thickness 0.254) (filled_areas_thickness no)
+    (fill yes (thermal_gap 0.508) (thermal_bridge_width 0.508))
+    (polygon
+      (pts
+        (xy 154.813 96.393)
+        (xy 152.527 96.393)
+        (xy 152.527 94.107)
+        (xy 154.813 94.107)
+      )
+    )
+  )
+  (zone (net 0) (net_name "") (layer "F.Cu") (hatch edge 0.508)
     (connect_pads yes (clearance 0.127))
     (min_thickness 0.127) (filled_areas_thickness no)
@@
   )
   (zone (net 0) (net_name "") (layer "F.Cu") (hatch edge 0.508)
+    (connect_pads (clearance 0.127))
+    (min_thickness 0.254) (filled_areas_thickness no)
+    (fill yes (thermal_gap 0.508) (thermal_bridge_width 0.508))
+    (polygon
+      (pts
+        (xy 147.193 109.093)
+        (xy 144.907 109.093)
+        (xy 144.907 106.807)
+        (xy 147.193 106.807)
+      )
+    )
+  )
+  (zone (net 0) (net_name "") (layer "F.Cu") (hatch edge 0.508)
+    (connect_pads (clearance 0.127))
+    (min_thickness 0.254) (filled_areas_thickness no)
+    (fill yes (thermal_gap 0.508) (thermal_bridge_width 0.508))
+    (polygon
+      (pts
+        (xy 157.353 96.393)
+        (xy 155.067 96.393)
+        (xy 155.067 94.107)
+        (xy 157.353 94.107)
+      )
+    )
+  )
+  (zone (net 0) (net_name "") (layer "F.Cu") (hatch edge 0.508)
     (connect_pads yes (clearance 0.127))
     (min_thickness 0.127) (filled_areas_thickness no)
@@
   )
   (zone (net 0) (net_name "") (layer "F.Cu") (hatch edge 0.508)
+    (connect_pads (clearance 0.127))
+    (min_thickness 0.254) (filled_areas_thickness no)
+    (fill yes (thermal_gap 0.508) (thermal_bridge_width 0.508))
+    (polygon
+      (pts
+        (xy 157.353 109.093)
+        (xy 155.067 109.093)
+        (xy 155.067 106.807)
+        (xy 157.353 106.807)
+      )
+    )
+  )
+  (zone (net 0) (net_name "") (layer "F.Cu") (hatch edge 0.508)
     (connect_pads yes (clearance 0.127))
     (min_thickness 0.127) (filled_areas_thickness no)
@@
   )
   (zone (net 0) (net_name "") (layer "F.Cu") (hatch edge 0.508)
+    (connect_pads (clearance 0.127))
+    (min_thickness 0.254) (filled_areas_thickness no)
+    (fill yes (thermal_gap 0.508) (thermal_bridge_width 0.508))
+    (polygon
+      (pts
+        (xy 152.273 109.093)
+        (xy 149.987 109.093)
+        (xy 149.987 106.807)
+        (xy 152.273 106.807)
+      )
+    )
+  )
+  (zone (net 0) (net_name "") (layer "F.Cu") (hatch edge 0.508)
     (connect_pads yes (clearance 0.127))
     (min_thickness 0.127) (filled_areas_thickness no)
@@
   )
   (zone (net 0) (net_name "") (layer "F.Cu") (hatch edge 0.508)
+    (connect_pads (clearance 0.127))
+    (min_thickness 0.254) (filled_areas_thickness no)
+    (fill yes (thermal_gap 0.508) (thermal_bridge_width 0.508))
+    (polygon
+      (pts
+        (xy 144.653 109.093)
+        (xy 142.367 109.093)
+        (xy 142.367 106.807)
+        (xy 144.653 106.807)
+      )
+    )
+  )
+  (zone (net 0) (net_name "") (layer "F.Cu") (hatch edge 0.508)
     (connect_pads yes (clearance 0.127))
     (min_thickness 0.127) (filled_areas_thickness no)
@@
   )
   (zone (net 0) (net_name "") (layer "F.Cu") (hatch edge 0.508)
+    (connect_pads (clearance 0.127))
+    (min_thickness 0.254) (filled_areas_thickness no)
+    (fill yes (thermal_gap 0.508) (thermal_bridge_width 0.508))
+    (polygon
+      (pts
+        (xy 139.573 96.393)
+        (xy 137.287 96.393)
+        (xy 137.287 94.107)
+        (xy 139.573 94.107)
+      )
+    )
+  )
+  (zone (net 0) (net_name "") (layer "F.Cu") (hatch edge 0.508)
+    (connect_pads (clearance 0.127))
+    (min_thickness 0.254) (filled_areas_thickness no)
+    (fill yes (thermal_gap 0.508) (thermal_bridge_width 0.508))
+    (polygon
+      (pts
+        (xy 139.573 109.093)
+        (xy 137.287 109.093)
+        (xy 137.287 106.807)
+        (xy 139.573 106.807)
+      )
+    )
+  )
+  (zone (net 0) (net_name "") (layer "F.Cu") (hatch edge 0.508)
     (connect_pads yes (clearance 0.127))
     (min_thickness 0.127) (filled_areas_thickness no)
@@
     )
   )
+  (zone (net 0) (net_name "") (layer "F.Cu") (hatch edge 0.508)
+    (connect_pads (clearance 0.127))
+    (min_thickness 0.254) (filled_areas_thickness no)
+    (fill yes (thermal_gap 0.508) (thermal_bridge_width 0.508))
+    (polygon
+      (pts
+        (xy 142.113 109.093)
+        (xy 139.827 109.093)
+        (xy 139.827 106.807)
+        (xy 142.113 106.807)
+      )
+    )
+  )
+  (zone (net 0) (net_name "") (layer "F.Cu") (hatch edge 0.508)
+    (connect_pads (clearance 0.127))
+    (min_thickness 0.254) (filled_areas_thickness no)
+    (fill yes (thermal_gap 0.508) (thermal_bridge_width 0.508))
+    (polygon
+      (pts
+        (xy 144.653 96.393)
+        (xy 142.367 96.393)
+        (xy 142.367 94.107)
+        (xy 144.653 94.107)
+      )
+    )
+  )
+  (zone (net 0) (net_name "") (layer "F.Cu") (hatch edge 0.508)
+    (connect_pads (clearance 0.127))
+    (min_thickness 0.254) (filled_areas_thickness no)
+    (fill yes (thermal_gap 0.508) (thermal_bridge_width 0.508))
+    (polygon
+      (pts
+        (xy 149.733 96.393)
+        (xy 147.447 96.393)
+        (xy 147.447 94.107)
+        (xy 149.733 94.107)
+      )
+    )
+  )
+  (zone (net 0) (net_name "") (layer "F.Cu") (hatch edge 0.508)
+    (connect_pads (clearance 0.127))
+    (min_thickness 0.254) (filled_areas_thickness no)
+    (fill yes (thermal_gap 0.508) (thermal_bridge_width 0.508))
+    (polygon
+      (pts
+        (xy 147.193 96.393)
+        (xy 144.907 96.393)
+        (xy 144.907 94.107)
+        (xy 147.193 94.107)
+      )
+    )
+  )
+  (zone (net 0) (net_name "") (layer "F.Cu") (hatch edge 0.508)
+    (connect_pads (clearance 0.127))
+    (min_thickness 0.254) (filled_areas_thickness no)
+    (fill yes (thermal_gap 0.508) (thermal_bridge_width 0.508))
+    (polygon
+      (pts
+        (xy 152.273 96.393)
+        (xy 149.987 96.393)
+        (xy 149.987 94.107)
+        (xy 152.273 94.107)
+      )
+    )
+  )
+  (zone (net 0) (net_name "") (layer "F.Cu") (hatch edge 0.508)
+    (connect_pads (clearance 0.127))
+    (min_thickness 0.254) (filled_areas_thickness no)
+    (fill yes (thermal_gap 0.508) (thermal_bridge_width 0.508))
+    (polygon
+      (pts
+        (xy 142.113 96.393)
+        (xy 139.827 96.393)
+        (xy 139.827 94.107)
+        (xy 142.113 94.107)
+      )
+    )
+  )
   (zone (net 0) (net_name "") (layer "B.Mask") (hatch edge 0.508)
     (connect_pads (clearance 0.127))
@@
     (polygon
       (pts
-        (xy 157.607 106.807)
-        (xy 137.033 106.807)
-        (xy 137.033 96.393)
-        (xy 157.607 96.393)
+        (xy 157.607 109.347)
+        (xy 137.033 109.347)
+        (xy 137.033 93.853)
+        (xy 157.607 93.853)
       )
     )
@@
     (polygon
       (pts
-        (xy 157.607 106.807)
-        (xy 137.033 106.807)
-        (xy 137.033 96.393)
-        (xy 157.607 96.393)
-      )
-    )
+        (xy 157.607 109.347)
+        (xy 137.033 109.347)
+        (xy 137.033 93.853)
+        (xy 157.607 93.853)
+      )
+    )
