File: Passive Breakout/Passive Breakout.kicad_pcb (KiCad board)
At the start: 2 copper layers, 15.5 x 10.4 mm, 18 parts

Commit message: Updated Files
Parts:
- removed REF** (x5): R_0402_1005Metric, Resistor_SMD:R_0402_1005Metric
- removed REF** (x5): R_0603_1608Metric, Resistor_SMD:R_0603_1608Metric
- removed REF** (x2): C_0805_2012Metric, Capacitor_SMD:C_0805_2012Metric
- removed REF**: C_1206_3216Metric, Capacitor_SMD:C_1206_3216Metric
- removed REF** (x2): C_0402_1005Metric, Capacitor_SMD:C_0402_1005Metric
- removed REF** (x2): C_0603_1608Metric, Capacitor_SMD:C_0603_1608Metric
- removed REF**: R_0805_2012Metric, Resistor_SMD:R_0805_2012Metric
