File: SOIC-20 Breakout/SOIC-20 Breakout.kicad_pcb (KiCad board)
At the start: 2 copper layers, 25.7 x 25.7 mm, 4 parts

Commit message: Updated files
Parts:
- added REF**: C_0603_1608Metric, Capacitor_SMD:C_0603_1608Metric, F.Cu at (162.6, 100.3)
Other:
- board size 25.7 x 25.7 mm -> 23.1 x 28.2 mm

Commit message: Updated Files
Parts:
- removed REF**: SOIC-20W_7.5x12.8mm_P1.27mm, Package_SO:SOIC-20W_7.5x12.8mm_P1.27mm
- removed REF**: SOIC-16_3.9x9.9mm_P1.27mm, Package_SO:SOIC-16_3.9x9.9mm_P1.27mm
- removed REF**: C_0603_1608Metric, Capacitor_SMD:C_0603_1608Metric
- removed REF**: MSOP-16_3x4mm_P0.5mm, Package_SO:MSOP-16_3x4mm_P0.5mm
- removed REF**: TSSOP-20_4.4x5mm_P0.5mm, Package_SO:TSSOP-20_4.4x5mm_P0.5mm
