File: SOIC-20 Breakout/SOIC-20 Breakout.kicad_pcb (KiCad board)
At the start: 2 copper layers, 23.1 x 28.2 mm, 0 parts

Commit message: Updated Files
Parts:
- added REF**: SOIC-20W_7.5x12.8mm_P1.27mm, Package_SO:SOIC-20W_7.5x12.8mm_P1.27mm, F.Cu at (152.4, 101.6)
Other:
- board size 23.1 x 28.2 mm -> 25.7 x 25.7 mm

Commit message: Updated files
Parts:
- added REF**: R_0603_1608Metric, Resistor_SMD:R_0603_1608Metric, B.Cu at (142.2, 90.2)
- added REF**: C_0603_1608Metric, Capacitor_SMD:C_0603_1608Metric, B.Cu at (157.5, 90.2)
- added REF**: C_0603_1608Metric, Capacitor_SMD:C_0603_1608Metric, B.Cu at (147.3, 113.0)
- added REF**: R_0603_1608Metric, Resistor_SMD:R_0603_1608Metric, B.Cu at (162.6, 113.0)
- added REF**: TSSOP-16_4.4x5mm_P0.65mm, Package_SO:TSSOP-16_4.4x5mm_P0.65mm, B.Cu at (152.4, 101.6)
- added REF**: R_0603_1608Metric, Resistor_SMD:R_0603_1608Metric, B.Cu at (142.2, 113.0)
- added REF**: C_0603_1608Metric, Capacitor_SMD:C_0603_1608Metric, B.Cu at (142.2, 100.3)
- added REF**: SOIC-16_3.9x9.9mm_P1.27mm, Package_SO:SOIC-16_3.9x9.9mm_P1.27mm, F.Cu at (152.4, 101.6)
- added REF**: R_0603_1608Metric, Resistor_SMD:R_0603_1608Metric, B.Cu at (162.6, 90.2)
- added REF**: C_0603_1608Metric, Capacitor_SMD:C_0603_1608Metric, B.Cu at (142.2, 102.9)
- added REF**: C_0603_1608Metric, Capacitor_SMD:C_0603_1608Metric, B.Cu at (147.3, 90.2)
- added REF**: TSSOP-20_4.4x6.5mm_P0.65mm, Package_SO:TSSOP-20_4.4x6.5mm_P0.65mm, B.Cu at (152.4, 101.6)
- added REF**: C_0603_1608Metric, Capacitor_SMD:C_0603_1608Metric, B.Cu at (162.6, 102.9)
- added REF**: C_0603_1608Metric, Capacitor_SMD:C_0603_1608Metric, B.Cu at (157.5, 113.0)
- added REF**: C_0603_1608Metric, Capacitor_SMD:C_0603_1608Metric, B.Cu at (162.6, 100.3)
