File: SOIC-20 Breakout/SOIC-20 Breakout.kicad_pcb (KiCad board)
At the start: 2 copper layers, 25.7 x 25.7 mm, 16 parts

Commit message: Updated Files
Parts:
- removed the REF** at (152.4, 101.6)
- moved REF** 1.91 mm to (155.6, 90.2)
- moved REF** 1.91 mm to (149.2, 113.0)
- moved REF** 1.91 mm to (160.7, 113.0)
- moved REF** 1.91 mm to (144.1, 113.0)
- moved REF** 1.91 mm to (144.1, 100.3)
- moved REF** 1.91 mm to (160.7, 90.2)
- moved REF** 1.91 mm to (144.1, 102.9)
- moved REF** 1.91 mm to (149.2, 90.2)
- moved REF** 1.91 mm to (160.7, 102.9)
- moved REF** 1.91 mm to (155.6, 113.0)
- moved REF** 1.91 mm to (160.7, 100.3)
- moved REF** 1.91 mm to (144.1, 90.2)
Other:
- board size 25.7 x 25.7 mm -> 21.8 x 25.7 mm
